File: kicad/inkkeys.kicad_pcb (KiCad board)
At the start: 2 copper layers, 110 x 50 mm, 60 parts, among them J1 Conn_01x07, SW1 SW_Push, SW10 SW_Push, SW11 Rotary_Encoder_Switch, SW12 SW_MEC_5G, SW13 SW_DPST_x2, SW2 SW_Push, SW3 SW_Push, SW4 SW_Push, SW5 SW_Push, SW6 SW_Push, SW7 SW_Push, SW8 SW_Push, SW9 SW_Push

Commit message: PCB Work
Parts:
- removed D26: WS2812B, LED_SMD:LED_WS2812B_PLCC4_5.0x5.0mm_P3.2mm
- removed SW11: Rotary_Encoder_Switch, Rotary_Encoder:RotaryEncoder_Alps_EC11E-Switch_Vertical_H20mm
- added J2: Conn_01x05, Connector_PinHeader_2.54mm:PinHeader_1x05_P2.54mm_Horizontal, F.Cu at (183.0, 71.0)
- added J3: Conn_01x03, Connector_PinHeader_2.54mm:PinHeader_1x03_P2.54mm_Horizontal, F.Cu at (197.0, 79.0)
- B1, C3, C4, D11, D14, D17, D20, D23: moved to B.Cu
- C1, C2: footprint Capacitor_THT:C_Disc_D5.0mm_W2.5mm_P5.00mm -> Capacitor_SMD:C_1206_3216Metric_Pad1.33x1.80mm_HandSolder
- moved D10 148.6 mm to (186.8, 113.0), turned to 270 degrees
- moved D25 148.2 mm to (190.5, 130.5)
- moved D9 141.0 mm to (186.8, 105.5), turned to 90 degrees
- moved D24 138.4 mm to (190.5, 90.5)
- moved D11 138.3 mm to (202.0, 134.0)
- moved D14 137.9 mm to (202.0, 66.0)
- moved C2 125.2 mm to (188.0, 77.0), turned to 270 degrees
- moved D8 120.9 mm to (167.8, 113.0), turned to 270 degrees
- moved C4 120.1 mm to (194.0, 77.0), turned to 90 degrees
- moved C1 118.5 mm to (183.0, 77.0), turned to 270 degrees
- moved R6 114.5 mm to (180.5, 77.0), turned to 270 degrees
- moved R8 113.6 mm to (185.5, 77.0), turned to 270 degrees
- moved D7 112.2 mm to (167.8, 105.5), turned to 90 degrees
- moved D21 111.0 mm to (171.5, 90.5)
- moved D23 110.5 mm to (154.0, 110.0)
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Connections:
- net /WS2812Bs/DOUT renamed Net-(D11-Pad4)
- net Net-(C1-Pad1) renamed /RA
- net Net-(C2-Pad1) renamed /RC
- B1 pad 20: Net-(B1-Pad20) -> /RS1
Routing:
- net +5V: track 0.00 -> 150.0 mm, vias 0 -> 2
- net Net-(D14-Pad1): track 0.00 -> 99.0 mm
- net Net-(D13-Pad4): track 0.00 -> 89.9 mm
- net /Row2: track 0.00 -> 81.5 mm
- net /Row1: track 0.00 -> 76.2 mm
- net Net-(D20-Pad1): track 0.00 -> 76.0 mm, vias 0 -> 2
- net Net-(D17-Pad1): track 0.00 -> 74.3 mm
- net Net-(D11-Pad1): track 0.00 -> 70.0 mm
- net /RS1: track 0.00 -> 51.4 mm, vias 0 -> 3
- net Net-(B1-Pad1): track 0.00 -> 30.8 mm
- net Net-(D18-Pad1): track 0.00 -> 28.0 mm
- net Net-(D15-Pad1): track 0.00 -> 27.6 mm
- net Net-(D22-Pad1): track 0.00 -> 24.7 mm
- net Net-(D16-Pad1): track 0.00 -> 24.7 mm
- net Net-(D13-Pad1): track 0.00 -> 24.7 mm
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- added copper zone on B.Cu, net GND
- added copper zone on F.Cu, net GND
Other:
- board size 110 x 50 mm -> 111 x 80 mm

Commit message: Logo and Credits
Parts:
- added G***: LOGO, inkkeys:hackropad, F.Cu at (172.0, 77.0)
Other:
- board text added: "Clement, Chris, Gabe, Hayley, Jack, Melinda, Nakul, & Parker Formlabs Hackathon 2021"

Commit message: Finished PCB and Generated Gerbers
Parts:
- added G***: LOGO, inkkeys:formlabslogo, F.Cu at (125.0, 78.5)
- SW12: value SW_MEC_5G -> SW_Push
- moved SW12 6.50 mm to (171.5, 64.5), turned to 180 degrees
- moved G*** 1.00 mm to (172.0, 76.0)
Connections:
- SW12 pad 2: Net-(B1-Pad22) -> GND
Routing:
- net /SLIDER_OUT: track 0.00 -> 81.3 mm, vias 0 -> 2
- net /Col1: track 7.01 -> 80.8 mm
- net Net-(D23-Pad1): track 0.00 -> 72.2 mm
- net /Col2: track 6.99 -> 52.0 mm, vias 0 -> 2
- net /Col5: track 7.01 -> 50.1 mm, vias 0 -> 3
- net /Row2: track 81.5 -> 119.9 mm, vias 0 -> 3
- net Net-(B1-Pad13): track 4.95 -> 41.1 mm
- net /RGB_D_OUT: track 0.00 -> 33.5 mm
- net /Row1: track 76.2 -> 109.4 mm
- net /OLED_CS: track 0.00 -> 31.7 mm
- net /OLED_DC: track 0.00 -> 30.9 mm
- net Net-(B1-Pad22): track 0.00 -> 30.2 mm
- net /Col3: track 6.97 -> 35.4 mm, vias 0 -> 2
- net /Col4: track 6.99 -> 34.1 mm, vias 0 -> 2
- net /OLED_RES: track 0.00 -> 25.1 mm, vias 0 -> 1
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- added copper zone on F.Cu, net +5V
- added copper zone on In2.Cu, net +5V
- added copper zone on In1.Cu, net GND
Other:
- copper layers 2 -> 4
- board text added: "Hackathon 2021"
- board text added: "LED Out"
- board text added: "OLED"
- board text added: "PWR SW"
- board text added: "RST"
- board text added: "Rotary Encoder"
- board text added: "Slider"
